File: KDT_Hierarchical.kicad_sch (KiCad schematic)
At the start: 0 parts

Commit message: init template
Other:
- removed sheet Power - Sequencing
- removed sheet Revision History
- note removed: "Power - Sequencing"
- note removed: "Revision History"
Changed lines of the file:
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@@
 		(effects
 			(font
-				(face "Times New Roman")
 				(size 4 4)
 				(color 0 0 0 1)
@@
 		)
 	)
-	(text "Power - Sequencing"
+	(text "..........................................."
 		(exclude_from_sim no)
 		(at 45.72 121.92 0)
 		(effects
 			(font
-				(face "Times New Roman")
 				(size 4 4)
 				(color 0 0 0 1)
@@
 		)
 	)
-	(text "Revision History"
+	(text "..........................................."
 		(exclude_from_sim no)
 		(at 45.72 129.54 0)
 		(effects
 			(font
-				(face "Times New Roman")
 				(size 4 4)
 				(color 0 0 0 1)
@@
 			(justify right bottom)
 			(href "#17")
-		)
-	)
-	(sheet
-		(at 340.36 313.69)
-		(size 35.56 5.08)
-		(stroke
-			(width 0.1524)
-			(type solid)
-		)
-		(fill
-			(color 0 0 0 0.0000)
-		)
-		(property "Sheetname" "Power - Sequencing"
-			(at 340.36 312.6609 0)
-			(effects
-				(font
-					(face "Times New Roman")
-					(size 1.905 1.905)
-					(bold yes)
-					(color 0 0 0 1)
-				)
-				(justify left bottom)
-			)
-		)
-		(property "Sheetfile" "Power - Sequencing.kicad_sch"
-			(at 341.63 314.96 0)
-			(effects
-				(font
-					(face "Arial")
-					(size 1.27 1.27)
-				)
-				(justify left top)
-			)
-		)
-		(instances
-			(project "KDT_Hierarchical"
-				(path "/0650c7a8-acba-429c-9f8e-eec0baf0bc1c"
-					(page "6")
-				)
-			)
 		)
 	)
@@
 				)
 			)
-		)
-	)
-	(sheet
-		(at 340.36 302.26)
-		(size 35.56 5.08)
-		(stroke
-			(width 0)
-			(type solid)
-		)
-		(fill
-			(color 0 0 0 0.0000)
-		)
-		(property "Sheetname" "Revision History"
-			(at 340.36 300.99 0)
-			(effects
-				(font
-					(face "Times New Roman")
-					(size 1.905 1.905)
-					(bold yes)
-					(color 0 0 0 1)
-				)
-				(justify left bottom)
-			)
-		)
-		(property "Sheetfile" "Revision History.kicad_sch"
-			(at 340.995 303.53 0)
-			(effects
-				(font
-					(face "Arial")
-					(size 1.27 1.27)
-				)
-				(justify left top)
-			)
-		)
-		(instances
-			(project "KDT_Hierarchical"
-				(path "/0650c7a8-acba-429c-9f8e-eec0baf0bc1c"
-					(page "7")
-				)
-			)
